File: laserradio/laserradio.kicad_sch (KiCad schematic)
At the start: 89 parts, among them J1 USB4105-GF-A, J3 DEBUG, J4 RIGHT, SW1 SW_SPDT, SW2 SW_SPDT, U1 W25Q128JV, U2 RP2040, U3 MCP1702T-3302E_CB, U4 ADA4891, U5 RS2255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

Commit message: WIP
Parts:
- removed D1: LED, LED_SMD:LED_0805_2012Metric, symbol Device:LED_Filled
- removed R7: 1K, Resistor_SMD:R_0603_1608Metric, symbol Device:R
- J4: footprint Connector_PinHeader_2.54mm:PinHeader_1x20_P2.54mm_Vertical -> Connector_PinHeader_2.54mm:PinHeader_1x15_P2.54mm_Vertical; symbol Connector_Generic:Conn_01x20 -> Connector_Generic:Conn_01x15
Connections:
- net GND: now also J4.14 (Pin_14); no longer J4.19 (Pin_19)
- net GPIO16: no longer J4.18 (Pin_18)
- net GPIO17: no longer J4.17 (Pin_17)
- net GPIO18: no longer J4.16 (Pin_16)
- net GPIO19: no longer J4.15 (Pin_15)
- net GPIO20: no longer J4.14 (Pin_14)
- net RUN: now also J4.15 (Pin_15); no longer J4.20 (Pin_20)
- no-connect marks 9 -> 15

Commit message: change resistor values to match what we have in stock
Parts:
- R10: value 330k -> 316k
- R13, R17: value 1k -> 1K
- R19, R32: value 5k -> 4.99k
- R24: value 1.2k -> 1.1k
- R5, R6: value 27Ω -> 30
Changed lines of the file:
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@@
     (in_bom yes) (on_board yes)
     (property "Reference" "R6" (id 0) (at 72.39 46.99 90))
-    (property "Value" "27Ω" (id 1) (at 77.47 46.99 90))
+    (property "Value" "30" (id 1) (at 77.47 46.99 90))
     (property "Footprint" "Resistor_SMD:R_0603_1608Metric" (id 2) (at 74.93 51.308 90)
       (effects (font (size 1.27 1.27)) hide)
@@
     (in_bom yes) (on_board yes)
     (property "Reference" "R24" (id 0) (at 184.785 120.65 90))
-    (property "Value" "1.2k" (id 1) (at 184.785 125.73 90))
+    (property "Value" "1.1k" (id 1) (at 184.785 125.73 90))
     (property "Footprint" "Resistor_SMD:R_0603_1608Metric" (id 2) (at 184.785 124.968 90)
       (effects (font (size 1.27 1.27)) hide)
@@
     (in_bom yes) (on_board yes)
     (property "Reference" "R32" (id 0) (at 256.54 135.89 0))
-    (property "Value" "5k" (id 1) (at 256.54 133.35 0))
+    (property "Value" "4.99k" (id 1) (at 256.54 133.35 0))
     (property "Footprint" "Resistor_SMD:R_0603_1608Metric" (id 2) (at 255.143 134.62 90)
       (effects (font (size 1.27 1.27)) hide)
@@
     (in_bom yes) (on_board yes)
     (property "Reference" "R5" (id 0) (at 72.39 41.91 90))
-    (property "Value" "27Ω" (id 1) (at 77.47 41.91 90))
+    (property "Value" "30" (id 1) (at 77.47 41.91 90))
     (property "Footprint" "Resistor_SMD:R_0603_1608Metric" (id 2) (at 74.93 46.228 90)
       (effects (font (size 1.27 1.27)) hide)
@@
       (effects (font (size 1.27 1.27)) (justify left))
     )
-    (property "Value" "5k" (id 1) (at 226.06 132.7149 0)
+    (property "Value" "4.99k" (id 1) (at 226.06 132.7149 0)
       (effects (font (size 1.27 1.27)) (justify left))
     )
@@
     (in_bom yes) (on_board yes)
     (property "Reference" "R13" (id 0) (at 236.855 62.23 90))
-    (property "Value" "1k" (id 1) (at 236.855 67.31 90))
+    (property "Value" "1K" (id 1) (at 236.855 67.31 90))
     (property "Footprint" "Resistor_SMD:R_0603_1608Metric" (id 2) (at 236.855 66.548 90)
       (effects (font (size 1.27 1.27)) hide)
@@
       (effects (font (size 1.27 1.27)) (justify left))
     )
-    (property "Value" "330k" (id 1) (at 233.68 40.6399 0)
+    (property "Value" "316k" (id 1) (at 233.68 40.6399 0)
       (effects (font (size 1.27 1.27)) (justify left))
     )
@@
     (in_bom yes) (on_board yes)
     (property "Reference" "R17" (id 0) (at 331.47 143.51 90))
-    (property "Value" "1k" (id 1) (at 336.55 143.51 90))
+    (property "Value" "1K" (id 1) (at 336.55 143.51 90))
     (property "Footprint" "Resistor_SMD:R_0603_1608Metric" (id 2) (at 335.788 143.51 90)
       (effects (font (size 1.27 1.27)) hide)
@@
     )
     (path "/7f6a80c7-dc6b-4786-9952-60d3f88f3192"
-      (reference "R5") (unit 1) (value "27Ω") (footprint "Resistor_SMD:R_0603_1608Metric")
+      (reference "R5") (unit 1) (value "30") (footprint "Resistor_SMD:R_0603_1608Metric")
     )
     (path "/1308c451-0f58-4964-928c-da3a6a9b1f5b"
-      (reference "R6") (unit 1) (value "27Ω") (footprint "Resistor_SMD:R_0603_1608Metric")
+      (reference "R6") (unit 1) (value "30") (footprint "Resistor_SMD:R_0603_1608Metric")
     )
     (path "/cae10f5e-e5a0-4e05-aa2b-158047ba406b"
@@
     )
     (path "/ba6c7f1c-2571-43fb-89b7-6e02955014c3"
-      (reference "R10") (unit 1) (value "330k") (footprint "Resistor_SMD:R_0603_1608Metric")
+      (reference "R10") (unit 1) (value "316k") (footprint "Resistor_SMD:R_0603_1608Metric")
     )
     (path "/5266eb3d-5bed-404c-b16f-d86c174f46eb"
@@
     )
     (path "/a9a43413-5ae2-4d2c-927c-c74d6e6a7481"
-      (reference "R13") (unit 1) (value "1k") (footprint "Resistor_SMD:R_0603_1608Metric")
+      (reference "R13") (unit 1) (value "1K") (footprint "Resistor_SMD:R_0603_1608Metric")
     )
     (path "/748fb544-91be-4cfa-b5cc-93dea8feef2a"
@@
     )
     (path "/baf95843-708a-4635-889c-12182973a39e"
-      (reference "R17") (unit 1) (value "1k") (footprint "Resistor_SMD:R_0603_1608Metric")
+      (reference "R17") (unit 1) (value "1K") (footprint "Resistor_SMD:R_0603_1608Metric")
     )
     (path "/4f1222a4-3c40-438c-89e3-c6f80473ae11"
@@
     )
     (path "/884e42e4-e625-4ead-b2f4-7cc51e5fa481"
-      (reference "R19") (unit 1) (value "5k") (footprint "Resistor_SMD:R_0603_1608Metric")
+      (reference "R19") (unit 1) (value "4.99k") (footprint "Resistor_SMD:R_0603_1608Metric")
     )
     (path "/e656eeff-6e08-4f0b-ad4a-5763078166c6"
@@
     )
     (path "/18173bb0-4840-4390-be13-a0205acc6b9d"
-      (reference "R24") (unit 1) (value "1.2k") (footprint "Resistor_SMD:R_0603_1608Metric")
+      (reference "R24") (unit 1) (value "1.1k") (footprint "Resistor_SMD:R_0603_1608Metric")
     )
     (path "/e5e3bdb5-6e26-477c-824b-94db11b1d2f3"
@@
     )
     (path "/7ed0f30a-56dd-4307-a4b3-3b90d15db2b1"
-      (reference "R32") (unit 1) (value "5k") (footprint "Resistor_SMD:R_0603_1608Metric")
+      (reference "R32") (unit 1) (value "4.99k") (footprint "Resistor_SMD:R_0603_1608Metric")
     )
     (path "/953e8c6f-6f43-43b5-aad0-f05c0e1e28ff"

Commit message: add photodiode footprint
Parts:
- D4: footprint Eclectronics:Photodiode -> Eclectronics:Laser_photodiode_2_pad
Changed lines of the file:
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@@
     (property "Reference" "D4" (id 0) (at 161.6075 64.77 0))
     (property "Value" "D_Photo" (id 1) (at 161.6075 67.31 0))
-    (property "Footprint" "Eclectronics:Photodiode" (id 2) (at 161.925 71.12 0)
+    (property "Footprint" "Eclectronics:Laser_photodiode_2_pad" (id 2) (at 161.925 71.12 0)
       (effects (font (size 1.27 1.27)) hide)
     )
@@
     )
     (path "/36764396-eff8-4d03-b00d-4b63d469b7c7"
-      (reference "D4") (unit 1) (value "D_Photo") (footprint "Eclectronics:Photodiode")
+      (reference "D4") (unit 1) (value "D_Photo") (footprint "Eclectronics:Laser_photodiode_2_pad")
     )
     (path "/c3e4d23c-0631-4042-afe5-f6d6d5e0efee"
