File: laserradio2/laserradio2.kicad_sch (KiCad schematic)
At the start: 87 parts, among them J1 USB4105-GF-A, J3 DEBUG, J4 RIGHT, SW1 SW_SPDT, SW2 SW_SPDT, U1 W25Q128JV, U2 RP2040, U3 MCP1702T-3302E_CB, U4 ADA4891, U5 RS2255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

Commit message: Pushed final files
Parts:
- removed C24, C27, C28: 10pF, Capacitor_SMD:C_0603_1608Metric, symbol Device:C
- removed R24: 1.1k, Resistor_SMD:R_0603_1608Metric, symbol Device:R
- removed R25, R27, R28, R30: 3.3k, Resistor_SMD:R_0603_1608Metric, symbol Device:R
- removed R31: 20k, Resistor_SMD:R_0603_1608Metric, symbol Device:R
- removed RV2: Nominal 10k, Eclectronics:Laser Potentiometer, symbol Device:R_Potentiometer
- removed Rx-Center1: Conn_01x01_Female, Connector_PinHeader_2.54mm:PinHeader_1x01_P2.54mm_Vertical, symbol Connector:Conn_01x01_Female
- added POT: 1k, Resistor_SMD:R_0603_1608Metric, symbol Device:R
- C17: value 10pF -> 1pF
- C21: value 10pF -> 0.1uF
- R13: value 1K -> 10k
- R16: value 100k -> 3.16k
- R17: value 1K -> 10
- R26: value 3.3k -> 10M
- R29: value 3.3k -> 50k
Connections:
- net GND: now also POT.1
- net at Y2.3 (OUT): now also U6.10 (+)
- net at R29.1, U4.6 (-): now also POT.2
Other:
- note added: "Receiver (Final)"
- note added: "Transmitter (Final)"
- note removed: "Band Pass Filter [4.82MHz, 15.92MHz] Gain: 0.3030"
- note removed: "Receiver"
- note removed: "Transmitter"
- moved on the sheet: C15, C17, C18, C19, C20, C21, C22, C23, C25, D3, D4, LD1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
